Commit message: square path tracer & enable blades control & teleop

File: cfr_simulation/cfr_description/urdf/blades.urdf.xacro (robot description, xacro)
@@ -37,5 +37,5 @@
         <joint name="${prefix}front_blade_joint" type="continuous">
             <origin xyz="0.46 0 0" rpy="0 0 0" />
-            <parent link="base_link"/>
+            <parent link="base_footprint"/>
             <child link="${prefix}front_blade"/>
             <axis xyz="0 0 1" rpy="0 0 0" />
@@ -43,5 +43,5 @@
         <joint name="${prefix}rear_blade_joint" type="continuous">
             <origin xyz="-0.46 0 0" rpy="0 0 0" />
-            <parent link="base_link"/>
+            <parent link="base_footprint"/>
             <child link="${prefix}rear_blade"/>
             <axis xyz="0 0 1" rpy="0 0 0" />

File: cfr_simulation/cfr_description/urdf/cfr_description.urdf.xacro (robot description, xacro)
@@ -72,5 +72,5 @@
                 <publish_odom>true</publish_odom>
                 <publish_odom_tf>true</publish_odom_tf>
-                <robotBaseFrame>cfr_link</robotBaseFrame>
+                <robotBaseFrame>base_footprint</robotBaseFrame>
             </plugin>
         </gazebo>

Commit message: add laser

File: cfr_simulation/cfr_description/urdf/blades.urdf.xacro (robot description, xacro)
@@ -28,14 +28,7 @@
           </visual>
         </link>
-        <!-- <gazebo reference="${prefix}_blade">
-            <mu1 value="1.0"/>
-            <mu2 value="0.5"/>
-            <kp value="100.0" />
-            <kd value="1.0" />
-            <fdir1 value="1 0 0"/>
-        </gazebo> -->
         <joint name="${prefix}front_blade_joint" type="continuous">
             <origin xyz="0.46 0 0" rpy="0 0 0" />
-            <parent link="base_footprint"/>
+            <parent link="base_link"/>
             <child link="${prefix}front_blade"/>
             <axis xyz="0 0 1" rpy="0 0 0" />
@@ -43,5 +36,5 @@
         <joint name="${prefix}rear_blade_joint" type="continuous">
             <origin xyz="-0.46 0 0" rpy="0 0 0" />
-            <parent link="base_footprint"/>
+            <parent link="base_link"/>
             <child link="${prefix}rear_blade"/>
             <axis xyz="0 0 1" rpy="0 0 0" />

File: cfr_simulation/cfr_description/urdf/cfr_description.urdf.xacro (robot description, xacro)
@@ -1,28 +1,27 @@
 <?xml version="1.0"?>
 <robot name="cfr" xmlns:xacro="http://ros.org/wiki/xacro">
+    <xacro:include filename="$(find cfr_description)/urdf/laser.urdf.xacro" />
+    <!-- 2D laser position -->
+    <xacro:property name="cfr_laser_dx" value="0.725" />
+    <xacro:property name="cfr_laser_dy" value="0.425" />
+    <xacro:property name="cfr_laser_dz" value="0.5" />
+    <xacro:property name="cfr_laser_yaw" value="${pi/4}" />
     <!-- Define robot constants -->
-    <xacro:property name="base_width" value="0.31"/>
-    <xacro:property name="base_length" value="0.42"/>
+    <xacro:property name="base_width" value="0.8"/>
+    <xacro:property name="base_length" value="1.6"/>
     <xacro:property name="base_height" value="0.18"/>
     <xacro:macro name="cfr" params="prefix">
         <!-- Robot Footprint -->
-        <link name="base_footprint">
-        </link>
+        <link name="base_footprint" />
         <!-- Robot Base -->
         <link name="base_link">
-            <collision>
-                <origin xyz="0 0 0" rpy="0 0 0"/>
+            <!-- <collision>
+                <origin xyz="0 0 0" rpy="0 0 ${pi/2}"/>
                 <geometry>
                   <box size="${base_length} ${base_width} ${base_height}"/>
                 </geometry>
-            </collision>
-            <!-- <visual>
-                <origin xyz="0 0 0" rpy="0 0 0"/>
-                <geometry>
-                  <box size="${base_length} ${base_width} ${base_height}"/>
-                </geometry>
-            </visual> -->
+            </collision> -->
             <inertial>
-                <origin xyz="0 0 1" rpy="0 0 0"/>
+                <origin xyz="0 0 0" rpy="0 0 ${pi/2}"/>
                 <mass value="1"/>
                 <inertia
@@ -35,5 +34,5 @@
             <parent link="base_footprint"/>
             <child link="base_link"/>
-            <origin xyz="0.0 0.0 0.0" rpy="0 0 0"/>
+            <origin xyz="0.0 0.0 0.0" rpy="0 0 ${pi/2}"/>
         </joint>
         <link name="cfr_link">
@@ -60,5 +59,5 @@
         </link>
         <joint name="cfr_joint" type="fixed">
-            <parent link="base_footprint"/>
+            <parent link="base_link"/>
             <child link="cfr_link"/>
             <origin xyz="0.0 0.0 0.0" rpy="0 0 0"/>
@@ -75,4 +74,16 @@
             </plugin>
         </gazebo>
+        <!-- <xacro:laser link="front_left_laser_link" />
+        <joint name="base_link_to_front_left_laser_joint" type="fixed">
+            <parent link="base_link" />
+            <child link="front_left_laser_link" />
+            <origin xyz="${cfr_laser_dx} ${-cfr_laser_dy} ${cfr_laser_dz}" rpy="0 0 ${-cfr_laser_yaw}" />
+        </joint>
+        <xacro:laser link="back_right_laser_link" />
+        <joint name="base_link_to_back_right_laser_joint" type="fixed">
+            <parent link="base_link" />
+            <child link="back_right_laser_link" />
+            <origin xyz="${-cfr_laser_dx} ${cfr_laser_dy} ${cfr_laser_dz}" rpy="0 0 ${cfr_laser_yaw+pi/2}" />
+        </joint> -->
     </xacro:macro>
 </robot>

Commit message: mesh rectification

File: cfr_simulation/cfr_description/urdf/blades.urdf.xacro (robot description, xacro)
@@ -2,5 +2,5 @@
 <robot name="cfr" xmlns:xacro="http://ros.org/wiki/xacro">
     <xacro:macro name="blades" params="prefix">
-        <link name="${prefix}front_blade">
+        <link name="${prefix}left_blade">
             <inertial>
               <mass value="0.01" />
@@ -9,11 +9,11 @@
             </inertial>
             <visual>
-              <origin xyz="-0.46 0 0" rpy="0 0 0" />
+              <origin xyz="-0.468 -0.002 0.05" rpy="0 0 0" />
               <geometry>
-                <mesh filename="file://$(find cfr_description)/meshes/CFR_blade_A.dae" />
+                <mesh filename="file://$(find cfr_description)/meshes/cfr_left_blade.dae" />
               </geometry>
             </visual>
         </link>
-        <link name="${prefix}rear_blade">
+        <link name="${prefix}right_blade">
           <inertial>
             <mass value="0.01" />
@@ -22,20 +22,20 @@
           </inertial>
           <visual>
-            <origin xyz="0.46 0 0" rpy="0 0 0" />
+            <origin xyz="0.468 -0.002 0.05" rpy="0 0 0" />
             <geometry>
-              <mesh filename="file://$(find cfr_description)/meshes/CFR_blade_B.dae" />
+              <mesh filename="file://$(find cfr_description)/meshes/cfr_right_blade.dae" />
             </geometry>
           </visual>
         </link>
-        <joint name="${prefix}front_blade_joint" type="continuous">
-            <origin xyz="0.46 0 0" rpy="0 0 0" />
+        <joint name="${prefix}left_blade_joint" type="continuous">
+            <origin xyz="0.468 0.002 0" rpy="0 0 0" />
             <parent link="base_link"/>
-            <child link="${prefix}front_blade"/>
+            <child link="${prefix}left_blade"/>
             <axis xyz="0 0 1" rpy="0 0 0" />
         </joint>
-        <joint name="${prefix}rear_blade_joint" type="continuous">
-            <origin xyz="-0.46 0 0" rpy="0 0 0" />
+        <joint name="${prefix}right_blade_joint" type="continuous">
+            <origin xyz="-0.468 0.002 0" rpy="0 0 0" />
             <parent link="base_link"/>
-            <child link="${prefix}rear_blade"/>
+            <child link="${prefix}right_blade"/>
             <axis xyz="0 0 1" rpy="0 0 0" />
         </joint>
@@ -44,5 +44,5 @@
                 <plugin>gazebo_ros2_control/GazeboSystem</plugin>
             </hardware>
-            <joint name="${prefix}front_blade_joint">
+            <joint name="${prefix}left_blade_joint">
               <command_interface name="velocity">
                 <param name="min">-120</param>
@@ -52,5 +52,5 @@
               <state_interface name="velocity"/>
             </joint>
-            <joint name="${prefix}rear_blade_joint">
+            <joint name="${prefix}right_blade_joint">
               <command_interface name="velocity">
                 <param name="min">120</param>

File: cfr_simulation/cfr_description/urdf/cfr_description.urdf.xacro (robot description, xacro)
@@ -50,7 +50,7 @@
             </collision>
             <visual>
-                <origin rpy="0 0 0" xyz="0 0 0"/>
+                <origin rpy="0 0 0" xyz="0 0 0.05"/>
                 <geometry>
-                    <mesh filename="file://$(find cfr_description)/meshes/CFR_body_without_blade.dae"/>
+                    <mesh filename="file://$(find cfr_description)/meshes/cfr_body_without_blades.dae"/>
                 </geometry>
             </visual>
