Commit message: fix laser

File: cfr_simulation/cfr_description/urdf/cfr_description.urdf.xacro (robot description, xacro)
@@ -16,10 +16,10 @@
         <!-- Robot Base -->
         <link name="base_link">
-            <!-- <collision>
-                <origin xyz="0 0 0" rpy="0 0 ${pi/2}"/>
+            <collision>
+                <origin xyz="0 0 0" rpy="0 0 0"/>
                 <geometry>
                   <box size="${base_length} ${base_width} ${base_height}"/>
                 </geometry>
-            </collision> -->
+            </collision>
             <inertial>
                 <origin xyz="0 0 0" rpy="0 0 ${pi/2}"/>
@@ -74,5 +74,5 @@
             </plugin>
         </gazebo>
-        <!-- <xacro:laser link="front_left_laser_link" />
+        <xacro:laser link="front_left_laser_link" />
         <joint name="base_link_to_front_left_laser_joint" type="fixed">
             <parent link="base_link" />
@@ -85,5 +85,5 @@
             <child link="back_right_laser_link" />
             <origin xyz="${-cfr_laser_dx} ${cfr_laser_dy} ${cfr_laser_dz}" rpy="0 0 ${cfr_laser_yaw+pi/2}" />
-        </joint> -->
+        </joint>
     </xacro:macro>
 </robot>

File: cfr_simulation/cfr_description/urdf/laser.urdf.xacro (robot description, xacro)
@@ -22,6 +22,6 @@
       </collision> -->
     </link>
-    <!-- <gazebo reference="${link}">
-      <sensor name="${link}" type="ray">
+    <gazebo reference="${link}">
+      <sensor name="${link}" type="gpu_ray">
         <always_on>true</always_on>
         <visualize>true</visualize>
@@ -55,5 +55,5 @@
         </plugin>
       </sensor>
-  </gazebo> -->
+  </gazebo>
   </xacro:macro>
 </robot>

Commit message: fix mesh collision ray bug

File: cfr_simulation/cfr_description/urdf/cfr_description.urdf.xacro (robot description, xacro)
@@ -8,7 +8,7 @@
     <xacro:property name="cfr_laser_yaw" value="${pi/4}" />
     <!-- Define robot constants -->
-    <xacro:property name="base_width" value="0.8"/>
-    <xacro:property name="base_length" value="1.6"/>
-    <xacro:property name="base_height" value="0.18"/>
+    <xacro:property name="base_width" value="1.0"/>
+    <xacro:property name="base_length" value="2.0"/>
+    <xacro:property name="base_height" value="0.4"/>
     <xacro:macro name="cfr" params="prefix">
         <!-- Robot Footprint -->
@@ -16,10 +16,16 @@
         <!-- Robot Base -->
         <link name="base_link">
-            <collision>
+            <!-- <visual>
+                <origin xyz="0 0 ${base_height/2}" rpy="0 0 0"/>
+                <geometry>
+                  <box size="${base_length} ${base_width} ${base_height}"/>
+                </geometry>
+            </visual> -->
+            <!-- <collision>
                 <origin xyz="0 0 0" rpy="0 0 0"/>
                 <geometry>
                   <box size="${base_length} ${base_width} ${base_height}"/>
                 </geometry>
-            </collision>
+            </collision> -->
             <inertial>
                 <origin xyz="0 0 0" rpy="0 0 ${pi/2}"/>
@@ -38,7 +44,7 @@
         <link name="cfr_link">
             <collision>
-                <origin rpy="0 0 0" xyz="0 0 0"/>
+                <origin rpy="0 0 0" xyz="0 0 ${base_height/2}"/>
                 <geometry>
-                    <mesh filename="file://$(find cfr_description)/meshes/CFR_body_without_blade.dae"/>
+                    <box size="${base_length} ${base_width} ${base_height}"/>
                 </geometry>
             </collision>

File: cfr_simulation/cfr_description/urdf/laser.urdf.xacro (robot description, xacro)
@@ -1,9 +1,4 @@
 <?xml version="1.0"?>
 <robot xmlns:xacro="http://ros.org/wiki/xacro">
-	<!-- lidar approximate physical properties -->
-  <!-- <xacro:property name="laser_x" value="0.08" />
-  <xacro:property name="laser_y" value="0.08" />
-  <xacro:property name="laser_z" value="0.12" />
-  <xacro:property name="laser_mass" value="0.5" /> -->
 	<!-- sick tim571 -->
   <xacro:macro name="laser" params="link">
@@ -23,8 +18,8 @@
     </link>
     <gazebo reference="${link}">
-      <sensor name="${link}" type="gpu_ray">
+      <sensor name="${link}" type="ray">
         <always_on>true</always_on>
         <visualize>true</visualize>
-        <update_rate>5</update_rate>
+        <update_rate>15</update_rate>
         <ray>
           <scan>

Commit message: Update new urdf and add cfr actuation joy param

File: cfr_simulation/cfr_description/urdf/cfr_description.urdf.xacro (robot description, xacro)
@@ -50,7 +50,8 @@
             </collision>
             <visual>
-                <origin rpy="0 0 0" xyz="0 0 0.05"/>
+                <origin rpy="${pi/2} 0 0" xyz="-0.0000 -0.01 0.05"/>
                 <geometry>
-                    <mesh filename="file://$(find cfr_description)/meshes/cfr_body_without_blades.dae"/>
+                    <!-- <mesh filename="file://$(find cfr_description)/meshes/cfr_body_without_blades.dae"/> -->
+                    <mesh filename="file://$(find cfr_description)/meshes/cfr_v2_body_without_blades.stl" scale="0.001 0.001 0.001"/>
                 </geometry>
             </visual>
@@ -84,5 +85,5 @@
             <parent link="base_link" />
             <child link="front_left_laser_link" />
-            <origin xyz="${cfr_laser_dx} ${-cfr_laser_dy} ${cfr_laser_dz}" rpy="0 0 ${-cfr_laser_yaw}" />
+            <origin xyz="${cfr_laser_dx} ${-cfr_laser_dy} ${cfr_laser_dz+0.05}" rpy="0 0 ${-cfr_laser_yaw}" />
         </joint>
         <xacro:laser link="back_right_laser_link" />
@@ -90,5 +91,5 @@
             <parent link="base_link" />
             <child link="back_right_laser_link" />
-            <origin xyz="${-cfr_laser_dx} ${cfr_laser_dy} ${cfr_laser_dz}" rpy="0 0 ${cfr_laser_yaw+pi/2}" />
+            <origin xyz="${-cfr_laser_dx} ${cfr_laser_dy} ${cfr_laser_dz+0.25}" rpy="0 0 ${cfr_laser_yaw+pi/2}" />
         </joint>
     </xacro:macro>
